Commit message: updated launch files and included new configurations for utm_auro experiments. Also updated xacro models to reduce laser min/max angle ranges and put hats on the robots so that they can see each other

File: urdf/materials.xacro (robot description, xacro)
@@ -25,3 +25,6 @@
 	  <color rgba="0.0 0.8 0.0 1.0"/>
   </material>
+	<material name="HatGrey">
+		<color rgba="0.1 0.1 0.1 1.0"/>
+	</material>
 </robot>

File: urdf/pioneer3dx.xacro (robot description, xacro)
@@ -312,4 +312,5 @@
 		<child link="back_sonar"/>
 	</joint>
+  <!-- Hokuyo Laser -->
   <joint name="hokuyo_joint" type="fixed">
     <origin xyz="0 0 0.085" rpy="0 0 0"/>
@@ -317,5 +318,4 @@
     <child link="laser"/>
   </joint>
-  <!-- Hokuyo Laser -->
   <link name="laser">
     <collision>
@@ -338,4 +338,5 @@
     </inertial>
   </link>
+  <!-- Camera -->
   <joint name="camera_joint" type="fixed">
     <origin xyz="0.17 0 0.0255" rpy="0 0 0"/>
@@ -343,5 +344,4 @@
     <child link="camera_link"/>
   </joint>
-  <!-- Camera -->
   <link name="camera_link">
     <collision>
@@ -357,4 +357,30 @@
       </geometry>
       <material name="CameraGreen"/>
+    </visual>
+    <inertial>
+      <mass value="1e-5" />
+      <origin xyz="0 0 0" rpy="0 0 0"/>
+      <inertia ixx="1e-6" ixy="0" ixz="0" iyy="1e-6" iyz="0" izz="1e-6" />
+    </inertial>
+  </link>
+  <!-- Hat -->
+  <joint name="hat_joint" type="fixed">
+    <origin xyz="0.0 0 0.0255" rpy="0 0 0"/>
+    <parent link="top_plate"/>
+    <child link="hat_link"/>
+  </joint>
+  <link name="hat_link">
+    <collision>
+      <origin xyz="0 0 0" rpy="0 0 0"/>
+      <geometry>
+	      <box size="0.15 0.2 0.4"/>
+      </geometry>
+    </collision>
+    <visual>
+      <origin xyz="0 0 0" rpy="0 0 0"/>
+      <geometry>
+      	<box size="0.15 0.2 0.4"/>
+      </geometry>
+      <material name="HatGrey"/>
     </visual>
     <inertial>
